File: Hardware/ebook_reader.brd (EAGLE design)
At the start: 170.2 x 111.2 mm, 103 parts, among them IC1 BD5229G-TR, IC4 XC6220A331MR-G, J1 FH34SRJ-24S-0.5SH_99_, J2 SAMACSYS_PARTS_USB4110-GF-A, J3 QWIIC_RIGHT_ANGLE, J4 112A-TAAR-R03_ATTEND, Q1 20V/4.2A/52mΩ/1.4W, Q2 20V/4.2A/52mΩ/1.4W, Q3 SI1308EDL-T1-GE3, U1 W25Q512JVEIQ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

Commit message: Issues fixed
Routing:
- net 3V3: track 440.8 -> 442.3 mm
Changed lines of the file:
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@@
 <wire x1="6.3" y1="48.5" x2="0" y2="48.5" width="0" layer="20"/>
 <wire x1="0" y1="48.5" x2="0" y2="0" width="0" layer="20"/>
+<dimension x1="0.1" y1="111.1" x2="22" y2="111.1" x3="11.05" y3="116" textsize="1.778" layer="1"/>
+<dimension x1="22" y1="110.2" x2="67" y2="110.2" x3="44.5" y3="123" textsize="1.778" layer="1"/>
+<dimension x1="67" y1="111.1" x2="91.580225" y2="111.199434375" x3="79.2582375" y3="119.029359375" textsize="1.778" layer="1"/>
+<dimension x1="92.21159375" y1="111.2" x2="92.212271875" y2="67.2" x3="159.000196875" y3="89.201028125" textsize="1.778" layer="1"/>
+<dimension x1="92.212271875" y1="67.2" x2="170.1" y2="67.3" x3="131.143628125" y3="76.991196875" textsize="1.778" layer="1"/>
+<dimension x1="170.1" y1="67.3" x2="170.2" y2="0.2" x3="192.976478125" y3="33.784015625" textsize="1.778" layer="1"/>
+<dimension x1="170.2" y1="0.2" x2="92" y2="0" x3="131.1308875" y3="-11.976646875" textsize="1.778" layer="1"/>
+<dimension x1="73.9" y1="9.9" x2="73.9" y2="0" x3="78" y3="4.95" textsize="1.778" layer="1"/>
+<dimension x1="92" y1="9.9" x2="73.9" y2="9.9" x3="82.95" y3="-7" textsize="1.778" layer="1"/>
+<dimension x1="73.9" y1="0" x2="0" y2="0" x3="36.95" y3="-12" textsize="1.778" layer="1"/>
+<dimension x1="0" y1="0" x2="0" y2="48.5" x3="-28" y3="24.25" textsize="1.778" layer="1"/>
+<dimension x1="0.1" y1="66.5" x2="0.1" y2="111.1" x3="-28" y3="88.8" textsize="1.778" layer="1"/>
+<dimension x1="6.3" y1="48.5" x2="6.3" y2="66.4" x3="-28" y3="57.45" textsize="1.778" layer="1"/>
 </plain>
 <attributes>
@@
 </class>
 </classes>
-<designrules name="jlcpcb-2layers.dru">
+<designrules name="jlcpcb-2layers.dru *">
 <param name="mdWireWire" value="5mil"/>
 <param name="mdWirePad" value="5mil"/>
@@
 <wire x1="5.7785" y1="89.281" x2="5.72" y2="89.22" width="0.3" layer="1"/>
 <wire x1="9" y1="101.25" x2="9.0805" y2="101.177584375" width="0.3" layer="1"/>
-<wire x1="35.1155" y1="100.0125" x2="41.656" y2="100.0125" width="0.3" layer="1"/>
-<wire x1="41.656" y1="100.0125" x2="48.1965" y2="100.0125" width="0.3" layer="1"/>
-<wire x1="27.4955" y1="107.6325" x2="35.1155" y2="100.0125" width="0.3" layer="1"/>
-<wire x1="48.1965" y1="100.0125" x2="48.31" y2="99.94" width="0.3" layer="1"/>
+<wire x1="27.4955" y1="107.6325" x2="39.656" y2="95.472" width="0.3" layer="1"/>
 <wire x1="27.4955" y1="107.6325" x2="27.38" y2="107.74" width="0.3" layer="1"/>
 <wire x1="35.7505" y1="56.642" x2="35.7505" y2="56.4515" width="0.3" layer="1"/>
@@
 <wire x1="84.328" y1="46.736" x2="84.22" y2="46.78" width="0.3" layer="1"/>
 <wire x1="118.999" y1="41.91" x2="119.15" y2="41.9" width="0.3" layer="1"/>
-<wire x1="41.656" y1="59.4995" x2="41.656" y2="100.0125" width="0.3" layer="1"/>
+<wire x1="41.656" y1="59.4995" x2="41.656" y2="96.4777375" width="0.3" layer="1"/>
+<wire x1="39.656" y1="95.472" x2="39.656" y2="94.4777375" width="0.3" layer="1"/>
 <wire x1="9.017" y1="63.373" x2="9.017" y2="48.8315" width="0.3" layer="1"/>
 <wire x1="7.0485" y1="65.3415" x2="9.017" y2="63.373" width="0.3" layer="1"/>
@@
 <wire x1="6.8847375" y1="89.247" x2="7.447" y2="88.6847375" width="0.3" layer="1"/>
 <wire x1="7.447" y1="88.6847375" x2="7.447" y2="86.6315" width="0.3" layer="1"/>
+<wire x1="48.31" y1="99.94" x2="47.937" y2="99.567" width="0.3" layer="1"/>
+<wire x1="47.937" y1="99.567" x2="44.7452625" y2="99.567" width="0.3" layer="1"/>
+<wire x1="44.7452625" y1="99.567" x2="41.656" y2="96.4777375" width="0.3" layer="1"/>
+<wire x1="39.656" y1="94.4777375" x2="41.656" y2="96.4777375" width="0.3" layer="1"/>
 </signal>
 <signal name="SS_SD" class="1">
@@
 <wire x1="48.26" y1="100.838" x2="47.9425" y2="100.5205" width="0.15" layer="1"/>
 <wire x1="10.414" y1="48.7045" x2="10.362" y2="48.702" width="0.15" layer="1"/>
-<wire x1="48.26" y1="100.838" x2="48.31" y2="100.89" width="0.15" layer="1"/>
+<wire x1="48.31" y1="100.89" x2="48.26" y2="100.838" width="0.15" layer="1"/>
 <wire x1="62.23" y1="109.474" x2="65.659" y2="109.474" width="0.15" layer="1"/>
 <wire x1="65.659" y1="109.474" x2="65.69" y2="109.475" width="0.15" layer="1"/>
@@
 <wire x1="45.6565" y1="109.1565" x2="45.6" y2="109.15" width="0.15" layer="1"/>
 <wire x1="47.244" y1="109.474" x2="47.29" y2="109.475" width="0.15" layer="1"/>
-<wire x1="14.224" y1="68.199" x2="14.224" y2="66.2305" width="0.15" layer="1"/>
-<wire x1="41.148" y1="95.123" x2="14.224" y2="68.199" width="0.15" layer="1"/>
+<wire x1="14.224" y1="66.2305" x2="14.224" y2="68.199" width="0.15" layer="1"/>
+<wire x1="14.224" y1="68.199" x2="41.148" y2="95.123" width="0.15" layer="1"/>
 <wire x1="41.148" y1="104.648" x2="41.148" y2="95.123" width="0.15" layer="16"/>
 <wire x1="44.7675" y1="108.2675" x2="41.148" y2="104.648" width="0.15" layer="16"/>
 <wire x1="45.593" y1="109.093" x2="44.7675" y2="108.2675" width="0.15" layer="1"/>
-<wire x1="14.224" y1="66.2305" x2="14.172" y2="66.202" width="0.15" layer="1"/>
+<wire x1="14.172" y1="66.202" x2="14.224" y2="66.2305" width="0.15" layer="1"/>
 <wire x1="45.593" y1="109.093" x2="45.6" y2="109.15" width="0.15" layer="1"/>
 <wire x1="47.3075" y1="109.474" x2="50.7365" y2="109.474" width="0.15" layer="1"/>
