File: Hardware/ebook_reader.sch (EAGLE design)
At the start: 103 parts, among them IC1 BD5229G-TR, IC4 XC6220A331MR-G, J1 FH34SRJ-24S-0.5SH_99_, J2 SAMACSYS_PARTS_USB4110-GF-A, J3 QWIIC_RIGHT_ANGLE, J4 112A-TAAR-R03_ATTEND, Q1 20V/4.2A/52mΩ/1.4W, Q2 20V/4.2A/52mΩ/1.4W, Q3 SI1308EDL-T1-GE3, U1 W25Q512JVEIQ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

Commit message: Issues fixed
Other:
- note added: "DMG2305UX-7"
- moved on the sheet: 3V3, D10, D11, D12, D6, D8, D9, EPD_3V3, EPD_3V3_C, EPD_BUSY, EPD_DC, EPD_RST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
